File: PCB/smc.brd (EAGLE design)
At the start: 30 x 48 mm, 27 parts, among them IC1 ESP-12E/F

Commit message: ESP12
Parts:
- removed LDR-OUT: JST-XH-02-PIN-ROUND-PAD, Rembrandt Electronics - JST XH Connectors v1-0:JST-XH-02-PACKAGE-ROUND-PAD
- removed USB-C-CASE: 0, SparkFun:0603-RES
- added PWR: JST-XH-02-PIN-ROUND-PAD, Rembrandt Electronics - JST XH Connectors v1-0:JST-XH-02-PACKAGE-ROUND-PAD
- added U$2: MICROSD-PUSH-OUT, microsd:MICROSD-PUSH-OUT
- added U$3: 4PIN, mypad:4PIN
- added VSELECT: RES_SWITCH, switches:RES_SWITCH
- moved USE-DTR 11.5 mm to (21.4, 25.5), turned to 180 degrees
- moved LM1117 11.2 mm to (21.5, 18.0)
- moved U$1 9.00 mm to (24.0, 3.64)
- moved R1 9.00 mm to (18.1, 38.1)
- moved R3 8.95 mm to (15.5, 38.1)
- moved RST 7.60 mm to (24.4, 10.3), turned to 270 degrees
- moved 10V-100UF 5.58 mm to (13.5, 18.3), turned to 0 degrees
- moved R4 4.94 mm to (21.9, 25.0), flipped to the bottom, turned to 0 degrees
- moved R6 4.81 mm to (21.0, 38.1), turned to 90 degrees
- moved 5.1K1 4.68 mm to (20.2, 11.8)
- moved 5.1K2 4.68 mm to (20.2, 8.96)
- moved COM 3.00 mm to (27.2, 14.3)
- moved FLASH 3.00 mm to (27.2, 10.3)
- moved FLASH-BTN 0.91 mm to (11.1, 40.1)
- moved RST-BTN 0.91 mm to (4.90, 40.1)
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Connections:
- new net CLK: IC1.IO14, U$2.5
- new net IO10: IC1.IO10, LED.1
- new net IO9-CS: IC1.IO9, U$2.2
- new net MISO: IC1.IO12, R6.1, U$2.7
- new net MOSI: IC1.IO13, U$2.3
- new net N$16: IC1.ADC, LDR-IN.1, R7.1
- new net N$17: IC1.CS0, U$3.P4
- net 3V3: now also PWR.1, U$2.4, VSELECT.B
- net 5V: now also VSELECT.A; no longer COM.4
- net GND: now also PWR.2, U$1.SHIELD1, U$1.SHIELD2, U$1.SHIELD3, U$1.SHIELD4, U$2.6, U$2.G1, U$2.G2, U$2.G3, U$2.G4; no longer LDR-OUT.2, USB-C-CASE.2
- net N$10: now also IC1.MISO, U$3.P3; no longer IC1.IO14, LED.1
- net N$3: now also IC1.SCLK, U$3.P1; no longer IC1.IO12, LDR-IN.1, R7.1
- net N$4: now also COM.4, VSELECT.C; no longer IC1.IO13, LDR-OUT.1, R6.1
- net N$9: now also IC1.MOSI, U$3.P2; no longer U$1.SHIELD1, U$1.SHIELD2, U$1.SHIELD3, U$1.SHIELD4, USB-C-CASE.1
Routing:
- net MISO: track 0.00 -> 53.2 mm, vias 0 -> 2
- net N$4: track 61.1 -> 12.9 mm, vias 1 -> 0
- net MOSI: track 0.00 -> 41.7 mm, vias 0 -> 2
- net IO9-CS: track 0.00 -> 35.4 mm, vias 0 -> 2
- net CLK: track 0.00 -> 33.1 mm, vias 0 -> 1
- net N$16: track 0.00 -> 31.4 mm, vias 0 -> 2
- net N$3: track 37.2 -> 8.11 mm
- net IO10: track 0.00 -> 19.4 mm, vias 0 -> 1
- net N$8: track 4.40 -> 14.2 mm, vias 0 -> 1
- net RST: track 73.1 -> 65.1 mm, vias 2 -> 1
- net N$17: track 0.00 -> 7.67 mm, vias 0 -> 1
- net IO0: track 44.7 -> 37.3 mm
- net N$6: track 33.8 -> 27.2 mm, vias 2 -> 0
- net N$9: track 2.19 -> 8.52 mm, vias 0 -> 1
- net N$7: track 35.2 -> 28.9 mm
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
Commit message: add logo
Parts:
- renumbered C1 to C1-0.1UF, R1 to R1-10K, R2 to R2-10K, R3 to R3-10K, R4 to R4-10K, R5 to R5-10K, R6 to R6-10K, R7 to R7-10K, R8 to R8-330, U$2 to MICROSD
Connections:
- net 3V3: no longer LM1117.TAB
Routing:
- net 3V3: track 74.3 -> 70.0 mm
