File: PCB/smc.sch (EAGLE design)
At the start: 29 parts, among them IC1 ESP-12E/F

Commit message: add logo
Parts:
- renumbered C1 to C1-0.1UF, R1 to R1-10K, R2 to R2-10K, R3 to R3-10K, R4 to R4-10K, R5 to R5-10K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
Connections:
- net 3V3: no longer LM1117.OUT1
