File: PCB/smc2.brd (EAGLE design)
At the start: 30 x 48 mm, 27 parts, among them IC1 ESP-12E/F

Commit message: PCB v2
Parts:
- removed C1: 0.1uF, SparkFun:0603-CAP
- removed LDR-OUT: JST-XH-02-PIN-ROUND-PAD, Rembrandt Electronics - JST XH Connectors v1-0:JST-XH-02-PACKAGE-ROUND-PAD
- removed R1, R3, R4, R6: 10K, SparkFun:0603-RES
- removed R8: 330, SparkFun:0603-RES
- removed USB-C-CASE: 0, SparkFun:0603-RES
- added C1-0.1UF: 0.1uF, SparkFun:0603-CAP
- added PWR: JST-XH-02-PIN-ROUND-PAD, Rembrandt Electronics - JST XH Connectors v1-0:JST-XH-02-PACKAGE-ROUND-PAD
- added R1-10K, R3-10K, R4-10K: 10K, SparkFun:0603-RES
- added R8-330: 330, SparkFun:0603-RES
- added U$3: 4PIN, mypad:4PIN
- added VSELECT: RES_SWITCH, switches:RES_SWITCH
- moved 5.1K2 14.3 mm to (12.1, 14.4), turned to 90 degrees
- moved USE-DTR 11.5 mm to (21.4, 25.5), turned to 180 degrees
- moved LM1117 11.0 mm to (21.2, 18.0)
- moved 5.1K1 10.4 mm to (14.8, 14.3), turned to 90 degrees
- moved 10V-100UF 5.58 mm to (13.5, 18.3), turned to 0 degrees
- moved COM 3.00 mm to (27.2, 14.3)
- moved FLASH 3.00 mm to (27.2, 10.3)
- moved RST 2.69 mm to (27.2, 5.25), turned to 270 degrees
- moved FLASH-BTN 0.91 mm to (11.1, 40.1)
- moved RST-BTN 0.91 mm to (4.90, 40.1)
- moved IIC 0.68 mm to (9.94, 22.7)
- moved BUZZER 0.51 mm to (3.10, 22.7)
- flipped U$1 to the bottom
- renumbered R2 to R2-10K, R5 to R5-10K, R7 to R7-10K
Connections:
- new net IO10: IC1.IO10, LED.1
- new net N$16: IC1.ADC, LDR-IN.1, R7-10K.1
- new net N$17: IC1.CS0, U$3.P4
- net 3V3: now also C1-0.1UF.1, PWR.1, R1-10K.1, R3-10K.1, VSELECT.B; no longer C1.1, LM1117.TAB, R1.1, R3.1, R6.2
- net 5V: now also VSELECT.A; no longer COM.4
- net GND: now also C1-0.1UF.2, PWR.2, R4-10K.1, R8-330.1, U$1.SHIELD1, U$1.SHIELD2, U$1.SHIELD3, U$1.SHIELD4; no longer C1.2, LDR-OUT.2, R4.1, R8.1, USB-C-CASE.2
- net IO0: now also R3-10K.2; no longer R3.2
- net IO2: now also R1-10K.2; no longer R1.2
- net N$1: now also R4-10K.2; no longer R4.2
- net N$10: now also IC1.MISO, U$3.P3; no longer IC1.IO14, LED.1
- net N$3: now also IC1.SCLK, U$3.P1; no longer IC1.IO12, LDR-IN.1, R7-10K.1
- net N$4: now also COM.4, VSELECT.C; no longer IC1.IO13, LDR-OUT.1, R6.1
- net N$5: now also R8-330.2; no longer R8.2
- net N$9: now also IC1.MOSI, U$3.P2; no longer U$1.SHIELD1, U$1.SHIELD2, U$1.SHIELD3, U$1.SHIELD4, USB-C-CASE.1
Routing:
- net N$4: track 61.1 -> 12.9 mm, vias 1 -> 0
- net N$16: track 0.00 -> 40.4 mm, vias 0 -> 2
- net N$3: track 37.2 -> 8.11 mm
- net IO10: track 0.00 -> 16.3 mm, vias 0 -> 1
- net 3V3: track 74.8 -> 58.8 mm, vias 3 -> 1
- net N$8: track 4.40 -> 14.2 mm, vias 0 -> 1
- net N$17: track 0.00 -> 7.67 mm, vias 0 -> 1
- net IO0: track 44.7 -> 37.3 mm
- net N$6: track 33.8 -> 27.2 mm, vias 2 -> 0
- net N$9: track 2.19 -> 8.52 mm, vias 0 -> 1
- net N$7: track 35.2 -> 28.9 mm
- net RST: track 73.1 -> 68.2 mm, vias 2 -> 1
- net N$1: track 6.81 -> 2.89 mm, vias 1 -> 0
- net 5V: track 30.8 -> 34.5 mm
- net IO2: track 6.24 -> 9.75 mm
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