File: PCB/smc2.sch (EAGLE design)
At the start: 29 parts, among them IC1 ESP-12E/F

Commit message: PCB v2
Parts:
- removed R6: 10K, SparkFun:RESISTOR0603-RES
- removed U$2: MICROSD-PUSH-OUT, microsd:MICROSD-PUSH-OUT
- renumbered C1 to C1-0.1UF, R1 to R1-10K, R2 to R2-10K, R3 to R3-10K, R4 to R4-10K, R5 to R5-10K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
Connections:
- removed net CLK: IC1.IO14, U$2.CLK
- removed net IO9-CS: IC1.IO9, U$2.CD_DAT3_CS
- removed net MISO: IC1.IO12, R6.1, U$2.DAT0_DO
- removed net MOSI: IC1.IO13, U$2.CMD_DIN
- net 3V3: no longer LM1117.OUT1, R6.2, U$2.VDD
- net GND: no longer U$2.VSS
